File: mm_external_uart.kicad_sch (KiCad schematic)
At the start: 0 parts

Commit message: tp2
Parts:
- added C: 2.2uF, symbol Device:C
- added J4: Conn_01x04, symbol Connector_Generic:Conn_01x04
- added R: 100, symbol Device:R
Connections:
- new net: J4.3 (Pin_3), R.1
- new net +BATT: C.1, J4.2 (Pin_2)
- new net EXTERNAL_UART_RX: J4.4 (Pin_4)
- new net EXTERNAL_UART_TX: R.2
- new net GND: C.2, J4.1 (Pin_1)
Changed lines of the file:
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@@
 (kicad_sch (version 20230121) (generator eeschema)
   (paper "A4")
+  (wire (pts (xy 137.668 83.058) (xy 134.366 83.058))
+    (stroke (width 0) (type default))
+  )
+  (wire (pts (xy 134.62 85.598) (xy 137.668 85.598))
+    (stroke (width 0) (type default))
+  )
+  (wire (pts (xy 133.858 80.518) (xy 133.858 92.456))
+    (stroke (width 0) (type default))
+  )
+  (wire (pts (xy 134.366 83.058) (xy 134.366 72.136))
+    (stroke (width 0) (type default))
+  )
+  (wire (pts (xy 160.02 74.168) (xy 160.02 77.724))
+    (stroke (width 0) (type default))
+  )
+  (wire (pts (xy 160.02 61.722) (xy 160.02 66.548))
+    (stroke (width 0) (type default))
+  )
+  (wire (pts (xy 133.858 80.518) (xy 137.668 80.518))
+    (stroke (width 0) (type default))
+  )
+  (wire (pts (xy 123.698 85.598) (xy 127 85.598))
+    (stroke (width 0) (type default))
+  )
+  (wire (pts (xy 123.19 88.138) (xy 137.668 88.138))
+    (stroke (width 0) (type default))
+  )
+  (hierarchical_label "EXTERNAL_UART_TX" (shape output) (at 123.698 85.598 180) (fields_autoplaced)
+    (effects (font (size 1.27 1.27)) (justify right))
+  )
+  (hierarchical_label "EXTERNAL_UART_RX" (shape input) (at 123.19 88.138 180) (fields_autoplaced)
+    (effects (font (size 1.27 1.27)) (justify right))
+  )
+  (symbol (lib_id "power:GND") (at 133.858 92.456 0) (unit 1)
+    (in_bom yes) (on_board yes) (dnp no)
+    (property "Reference" "#PWR026" (at 133.858 98.806 0)
+      (effects (font (size 1.27 1.27)) hide)
+    )
+    (property "Value" "GND" (at 134.112 96.266 0)
+      (effects (font (size 1.27 1.27)))
+    )
+    (property "Footprint" "" (at 133.858 92.456 0)
+      (effects (font (size 1.27 1.27)) hide)
+    )
+    (property "Datasheet" "" (at 133.858 92.456 0)
+      (effects (font (size 1.27 1.27)) hide)
+    )
+    (pin "1")
+    (instances
+      (project "minimouse"
+        (path "/d8fa4cba-2469-4231-847f-065b6b829f44/d17bb1c7-f68a-465e-9a17-5858ef86fc30"
+          (reference "#PWR026") (unit 1)
+        )
+      )
+    )
+  )
+  (symbol (lib_id "Connector_Generic:Conn_01x04") (at 142.748 83.058 0) (unit 1)
+    (in_bom yes) (on_board yes) (dnp no) (fields_autoplaced)
+    (property "Reference" "J4" (at 144.78 83.058 0)
+      (effects (font (size 1.27 1.27)) (justify left))
+    )
+    (property "Value" "Conn_01x04" (at 144.78 85.598 0)
+      (effects (font (size 1.27 1.27)) (justify left))
+    )
+    (property "Footprint" "" (at 142.748 83.058 0)
+      (effects (font (size 1.27 1.27)) hide)
+    )
+    (property "Datasheet" "~" (at 142.748 83.058 0)
+      (effects (font (size 1.27 1.27)) hide)
+    )
+    (pin "3")
+    (pin "1")
+    (pin "4")
+    (pin "2")
+    (instances
+      (project "minimouse"
+        (path "/d8fa4cba-2469-4231-847f-065b6b829f44/d17bb1c7-f68a-465e-9a17-5858ef86fc30"
+          (reference "J4") (unit 1)
+        )
+      )
+    )
+  )
+  (symbol (lib_id "power:+BATT") (at 134.366 72.136 0) (unit 1)
+    (in_bom yes) (on_board yes) (dnp no) (fields_autoplaced)
+    (property "Reference" "#PWR027" (at 134.366 75.946 0)
+      (effects (font (size 1.27 1.27)) hide)
+    )
+    (property "Value" "+BATT" (at 134.366 67.056 0)
+      (effects (font (size 1.27 1.27)))
+    )
+    (property "Footprint" "" (at 134.366 72.136 0)
+      (effects (font (size 1.27 1.27)) hide)
+    )
+    (property "Datasheet" "" (at 134.366 72.136 0)
+      (effects (font (size 1.27 1.27)) hide)
+    )
+    (pin "1")
+    (instances
+      (project "minimouse"
+        (path "/d8fa4cba-2469-4231-847f-065b6b829f44/d17bb1c7-f68a-465e-9a17-5858ef86fc30"
+          (reference "#PWR027") (unit 1)
+        )
+      )
+    )
+  )
+  (symbol (lib_id "power:+BATT") (at 160.02 61.722 0) (unit 1)
+    (in_bom yes) (on_board yes) (dnp no) (fields_autoplaced)
+    (property "Reference" "#PWR014" (at 160.02 65.532 0)
+      (effects (font (size 1.27 1.27)) hide)
+    )
+    (property "Value" "+BATT" (at 160.02 56.642 0)
+      (effects (font (size 1.27 1.27)))
+    )
+    (property "Footprint" "" (at 160.02 61.722 0)
+      (effects (font (size 1.27 1.27)) hide)
+    )
+    (property "Datasheet" "" (at 160.02 61.722 0)
+      (effects (font (size 1.27 1.27)) hide)
+    )
+    (pin "1")
+    (instances
+      (project "minimouse"
+        (path "/d8fa4cba-2469-4231-847f-065b6b829f44/d17bb1c7-f68a-465e-9a17-5858ef86fc30"
+          (reference "#PWR014") (unit 1)
+        )
+      )
+    )
+  )
+  (symbol (lib_id "Device:C") (at 160.02 70.358 0) (unit 1)
+    (in_bom yes) (on_board yes) (dnp no) (fields_autoplaced)
+    (property "Reference" "C" (at 163.83 69.088 0)
+      (effects (font (size 1.27 1.27)) (justify left))
+    )
+    (property "Value" "2.2uF" (at 163.83 71.628 0)
+      (effects (font (size 1.27 1.27)) (justify left))
+    )
+    (property "Footprint" "" (at 160.9852 74.168 0)
+      (effects (font (size 1.27 1.27)) hide)
+    )
+    (property "Datasheet" "~" (at 160.02 70.358 0)
+      (effects (font (size 1.27 1.27)) hide)
+    )
+    (pin "2")
+    (pin "1")
+    (instances
+      (project "minimouse"
+        (path "/d8fa4cba-2469-4231-847f-065b6b829f44/d17bb1c7-f68a-465e-9a17-5858ef86fc30"
+          (reference "C") (unit 1)
+        )
+      )
+    )
+  )
+  (symbol (lib_id "Device:R") (at 130.81 85.598 270) (unit 1)
+    (in_bom yes) (on_board yes) (dnp no)
+    (property "Reference" "R" (at 129.54 80.772 90)
+      (effects (font (size 1.27 1.27)))
+    )
+    (property "Value" "100" (at 130.81 82.55 90)
+      (effects (font (size 1.27 1.27)))
+    )
+    (property "Footprint" "" (at 130.81 83.82 90)
+      (effects (font (size 1.27 1.27)) hide)
+    )
+    (property "Datasheet" "~" (at 130.81 85.598 0)
+      (effects (font (size 1.27 1.27)) hide)
+    )
+    (pin "2")
+    (pin "1")
+    (instances
+      (project "minimouse"
+        (path "/d8fa4cba-2469-4231-847f-065b6b829f44/d17bb1c7-f68a-465e-9a17-5858ef86fc30"
+          (reference "R") (unit 1)
+        )
+      )
+    )
+  )
+  (symbol (lib_id "power:GND") (at 160.02 77.724 0) (unit 1)
+    (in_bom yes) (on_board yes) (dnp no)
+    (property "Reference" "#PWR028" (at 160.02 84.074 0)
+      (effects (font (size 1.27 1.27)) hide)
+    )
+    (property "Value" "GND" (at 160.274 81.534 0)
+      (effects (font (size 1.27 1.27)))
+    )
+    (property "Footprint" "" (at 160.02 77.724 0)
+      (effects (font (size 1.27 1.27)) hide)
+    )
+    (property "Datasheet" "" (at 160.02 77.724 0)
+      (effects (font (size 1.27 1.27)) hide)
+    )
+    (pin "1")
+    (instances
+      (project "minimouse"
+        (path "/d8fa4cba-2469-4231-847f-065b6b829f44/d17bb1c7-f68a-465e-9a17-5858ef86fc30"
+          (reference "#PWR028") (unit 1)
+        )
+      )
+    )
+  )
 )

Commit message: TP3
Parts:
- C13: renamed from C; footprint (none) -> Capacitor_SMD:C_0603_1608Metric
- J4: footprint (none) -> Connector_PinHeader_2.54mm:PinHeader_1x04_P2.54mm_Vertical
- R17: renamed from R; footprint (none) -> Resistor_SMD:R_0603_1608Metric
Other:
- moved on the sheet: R17
Changed lines of the file:
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@@
     (stroke (width 0) (type default))
   )
-  (wire (pts (xy 134.62 85.598) (xy 137.668 85.598))
+  (wire (pts (xy 115.57 88.138) (xy 137.668 88.138))
     (stroke (width 0) (type default))
   )
-  (wire (pts (xy 133.858 80.518) (xy 133.858 92.456))
+  (wire (pts (xy 130.302 85.598) (xy 137.668 85.598))
+    (stroke (width 0) (type default))
+  )
+  (wire (pts (xy 131.572 80.518) (xy 131.572 92.456))
     (stroke (width 0) (type default))
   )
   (wire (pts (xy 134.366 83.058) (xy 134.366 72.136))
+    (stroke (width 0) (type default))
+  )
+  (wire (pts (xy 116.078 85.598) (xy 122.682 85.598))
     (stroke (width 0) (type default))
   )
@@
     (stroke (width 0) (type default))
   )
-  (wire (pts (xy 133.858 80.518) (xy 137.668 80.518))
+  (wire (pts (xy 131.572 80.518) (xy 137.668 80.518))
     (stroke (width 0) (type default))
   )
-  (wire (pts (xy 123.698 85.598) (xy 127 85.598))
-    (stroke (width 0) (type default))
-  )
-  (wire (pts (xy 123.19 88.138) (xy 137.668 88.138))
-    (stroke (width 0) (type default))
-  )
-  (hierarchical_label "EXTERNAL_UART_TX" (shape output) (at 123.698 85.598 180) (fields_autoplaced)
+  (hierarchical_label "EXTERNAL_UART_TX" (shape output) (at 116.078 85.598 180) (fields_autoplaced)
     (effects (font (size 1.27 1.27)) (justify right))
   )
-  (hierarchical_label "EXTERNAL_UART_RX" (shape input) (at 123.19 88.138 180) (fields_autoplaced)
+  (hierarchical_label "EXTERNAL_UART_RX" (shape input) (at 115.57 88.138 180) (fields_autoplaced)
     (effects (font (size 1.27 1.27)) (justify right))
   )
-  (symbol (lib_id "power:GND") (at 133.858 92.456 0) (unit 1)
+  (symbol (lib_id "power:GND") (at 131.572 92.456 0) (unit 1)
     (in_bom yes) (on_board yes) (dnp no)
-    (property "Reference" "#PWR026" (at 133.858 98.806 0)
+    (property "Reference" "#PWR026" (at 131.572 98.806 0)
       (effects (font (size 1.27 1.27)) hide)
     )
-    (property "Value" "GND" (at 134.112 96.266 0)
+    (property "Value" "GND" (at 131.826 96.266 0)
       (effects (font (size 1.27 1.27)))
     )
-    (property "Footprint" "" (at 133.858 92.456 0)
+    (property "Footprint" "" (at 131.572 92.456 0)
       (effects (font (size 1.27 1.27)) hide)
     )
-    (property "Datasheet" "" (at 133.858 92.456 0)
+    (property "Datasheet" "" (at 131.572 92.456 0)
       (effects (font (size 1.27 1.27)) hide)
     )
@@
       (effects (font (size 1.27 1.27)) (justify left))
     )
-    (property "Footprint" "" (at 142.748 83.058 0)
+    (property "Footprint" "Connector_PinHeader_2.54mm:PinHeader_1x04_P2.54mm_Vertical" (at 142.748 83.058 0)
       (effects (font (size 1.27 1.27)) hide)
     )
@@
   (symbol (lib_id "Device:C") (at 160.02 70.358 0) (unit 1)
     (in_bom yes) (on_board yes) (dnp no) (fields_autoplaced)
-    (property "Reference" "C" (at 163.83 69.088 0)
+    (property "Reference" "C13" (at 163.83 69.088 0)
       (effects (font (size 1.27 1.27)) (justify left))
     )
@@
       (effects (font (size 1.27 1.27)) (justify left))
     )
-    (property "Footprint" "" (at 160.9852 74.168 0)
+    (property "Footprint" "Capacitor_SMD:C_0603_1608Metric" (at 160.9852 74.168 0)
       (effects (font (size 1.27 1.27)) hide)
     )
@@
       (project "minimouse"
         (path "/d8fa4cba-2469-4231-847f-065b6b829f44/d17bb1c7-f68a-465e-9a17-5858ef86fc30"
-          (reference "C") (unit 1)
+          (reference "C13") (unit 1)
         )
       )
     )
   )
-  (symbol (lib_id "Device:R") (at 130.81 85.598 270) (unit 1)
+  (symbol (lib_id "Device:R") (at 126.492 85.598 270) (unit 1)
     (in_bom yes) (on_board yes) (dnp no)
-    (property "Reference" "R" (at 129.54 80.772 90)
+    (property "Reference" "R17" (at 124.206 81.026 90)
       (effects (font (size 1.27 1.27)))
     )
-    (property "Value" "100" (at 130.81 82.55 90)
+    (property "Value" "100" (at 125.476 82.804 90)
       (effects (font (size 1.27 1.27)))
     )
-    (property "Footprint" "" (at 130.81 83.82 90)
+    (property "Footprint" "Resistor_SMD:R_0603_1608Metric" (at 126.492 83.82 90)
       (effects (font (size 1.27 1.27)) hide)
     )
-    (property "Datasheet" "~" (at 130.81 85.598 0)
+    (property "Datasheet" "~" (at 126.492 85.598 0)
       (effects (font (size 1.27 1.27)) hide)
     )
@@
       (project "minimouse"
         (path "/d8fa4cba-2469-4231-847f-065b6b829f44/d17bb1c7-f68a-465e-9a17-5858ef86fc30"
-          (reference "R") (unit 1)
+          (reference "R17") (unit 1)
         )
       )
