File: mm_power.kicad_sch (KiCad schematic)
At the start: 1 part, among them J5 Conn_01x02

Commit message: tp2
Parts:
- added C (x2): 2.2uF, symbol Device:C
- added J6: Conn_01x02, Connector_PinHeader_2.54mm:PinHeader_1x02_P2.54mm_Vertical, symbol Connector_Generic:Conn_01x02
Connections:
- net +BATT: now also C.1
- net GND: now also C.2, C.2, J6.1 (Pin_1)
- new net +3.3V: C.1, J6.2 (Pin_2)

Commit message: TP3
Parts:
- removed J6: Conn_01x02, Connector_PinHeader_2.54mm:PinHeader_1x02_P2.54mm_Vertical, symbol Connector_Generic:Conn_01x02
- added D1: LED, LED_SMD:LED_0603_1608Metric, symbol Device:LED
- added R13: 330, Resistor_SMD:R_0603_1608Metric, symbol Device:R
- added U4: LP5907MFX-3.3, Package_TO_SOT_SMD:SOT-23-5, symbol Regulator_Linear:LP5907MFX-3.3
- C10, C11: renamed from C; footprint (none) -> Capacitor_SMD:C_0603_1608Metric
Connections:
- net +3.3V: now also R13.1, U4.5 (OUT)
- net +BATT: now also U4.1 (IN), U4.3 (EN)
- net GND: now also D1.1 (K), U4.2 (GND)
- new net: D1.2 (A), R13.2
Other:
- moved on the sheet: C11
