File: mm_motor_control.kicad_sch (KiCad schematic)
At the start: 0 parts

Commit message: tp2
Parts:
- added CEN: 10nF, symbol Device:C
- added CRCOFF: 22nf, symbol Device:C
- added CS: 2.2uF, symbol Device:C
- added CSTBY (x2): 1nF, symbol Device:C
- added R10, R11: R, symbol Device:R
- added REN, RSTBY: 18k, symbol Device:R
- added ROFF: 47k, symbol Device:R
- added RRCOFF: 1k, symbol Device:R
- added RSNSA, RSNSB: 330m, symbol Device:R
- added U3: STSPIN240, Package_DFN_QFN:VQFN-16-1EP_3x3mm_P0.5mm_EP1.8x1.8mm, symbol Driver_Motor:STSPIN240
Connections:
- net EN: now also REN.1
- net FAULT: now also CEN.1, REN.2, U3.13 (EN/FLT)
- net OUT_A1: now also U3.3 (OUTA1)
- net OUT_A2: now also U3.5 (OUTA2)
- net OUT_B1: now also U3.10 (OUTB1)
- net OUT_B2: now also U3.8 (OUTB2)
- net PHASE_A: now also U3.1 (PHA)
- net PHASE_B: now also U3.15 (PHB)
- net PWM_A: now also U3.2 (PWMA)
- net PWM_B: now also U3.16 (PWMB)
- net STBY/RESET: now also CSTBY.1, CSTBY.1, RSTBY.1, U3.14 (STBY/RESET)
- new net: ROFF.1, RRCOFF.1, U3.12 (TOFF)
- new net: CRCOFF.1, RRCOFF.2
- new net: CS.2, U3.6 (VS)
- new net: RSNSB.1, U3.9 (SENSEB)
- new net: R10.2, R11.1, U3.11 (REF)
- new net: RSNSA.1, U3.4 (SENSEA)
- new net +BATT: R10.1
- new net GND: CEN.2, CRCOFF.2, CS.1, CSTBY.2, CSTBY.2, R11.2, ROFF.2, RSNSA.2, RSNSB.2, U3.7 (GND)
- new net VDD: RSTBY.2

Commit message: TP3
Parts:
- removed CS: 2.2uF, symbol Device:C
- removed CSTBY (x2): 1nF, symbol Device:C
- removed RSTBY: 18k, symbol Device:R
- added C12: 2.2uF, Capacitor_SMD:C_0603_1608Metric, symbol Device:C
- CEN1: renamed from CEN; footprint (none) -> Capacitor_SMD:C_0603_1608Metric
- CRCOFF1: renamed from CRCOFF; footprint (none) -> Capacitor_SMD:C_0603_1608Metric
- R10, R11: value R -> 10k; footprint (none) -> Resistor_SMD:R_0603_1608Metric
- REN1: renamed from REN; value 18k -> 10k; footprint (none) -> Resistor_SMD:R_0603_1608Metric
- ROFF1: renamed from ROFF; footprint (none) -> Resistor_SMD:R_0603_1608Metric
- RRCOFF1: renamed from RRCOFF; footprint (none) -> Resistor_SMD:R_0603_1608Metric
- RSNSA1: renamed from RSNSA; footprint (none) -> Resistor_SMD:R_0603_1608Metric
- RSNSB1: renamed from RSNSB; footprint (none) -> Resistor_SMD:R_0603_1608Metric
Connections:
- net +BATT: now also U3.6 (VS), C12.1
- net GND: now also U3.17 (EPAD), C12.2
Other:
- moved on the sheet: CEN1, REN1

Commit message: fin de TP4
Connections:
- net GND: now also RSNSB1.1; no longer RSNSB1.2
- net at U3.9 (SENSEB): now also RSNSB1.2; no longer RSNSB1.1
Other:
- moved on the sheet: RSNSB1
Changed lines of the file:
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@@
     )
   )
-  (symbol (lib_id "Device:R") (at 167.64 100.33 0) (unit 1)
+  (symbol (lib_id "Device:R") (at 167.64 100.33 180) (unit 1)
     (in_bom yes) (on_board yes) (dnp no) (fields_autoplaced)
-    (property "Reference" "RSNSB1" (at 169.418 99.06 0)
-      (effects (font (size 1.27 1.27)) (justify left))
+    (property "Reference" "RSNSB1" (at 170.18 99.06 0)
+      (effects (font (size 1.27 1.27)) (justify right))
     )
-    (property "Value" "330m" (at 169.418 101.6 0)
-      (effects (font (size 1.27 1.27)) (justify left))
+    (property "Value" "330m" (at 170.18 101.6 0)
+      (effects (font (size 1.27 1.27)) (justify right))
     )
-    (property "Footprint" "Resistor_SMD:R_0603_1608Metric" (at 165.862 100.33 90)
+    (property "Footprint" "Resistor_SMD:R_0603_1608Metric" (at 169.418 100.33 90)
       (effects (font (size 1.27 1.27)) hide)
     )
