File: minimouse.kicad_pcb (KiCad board)
At the start: 2 copper layers, 90 x 85 mm, 22 parts, among them J1 Conn_ARM_JTAG_SWD_10, J5 Conn_01x02, M1 N20_encoder, M2 N20_encoder, U1 STM32F030C8Tx, U4 HC-SR04

Commit message: TP3
Parts:
- added C10: 2.2uF, Capacitor_SMD:C_0603_1608Metric, F.Cu at (247.3, 70.8)
- added C11: 2.2uF, Capacitor_SMD:C_0603_1608Metric, F.Cu at (247.3, 73.3)
- added C12: 2.2uF, Capacitor_SMD:C_0603_1608Metric, F.Cu at (237.3, 70.8)
- added C13: 2.2uF, Capacitor_SMD:C_0603_1608Metric, F.Cu at (239.7, 97.5)
- added C7: 2.2uF, Capacitor_SMD:C_0603_1608Metric, F.Cu at (173.2, 92.6)
- added C8: 2.2uF, Capacitor_SMD:C_0603_1608Metric, F.Cu at (247.3, 80.3)
- added C9: 2.2uF, Capacitor_SMD:C_0603_1608Metric, F.Cu at (169.0, 78.4)
- added CEN1: 10nF, Capacitor_SMD:C_0603_1608Metric, F.Cu at (237.3, 73.3)
- added CRCOFF1: 22nf, Capacitor_SMD:C_0603_1608Metric, F.Cu at (237.3, 75.8)
- added D1: LED, LED_SMD:LED_0603_1608Metric, F.Cu at (167.0, 77.2)
- added J2: Conn_01x06, Connector_PinHeader_2.54mm:PinHeader_1x06_P2.54mm_Vertical, F.Cu at (179.0, 90.3)
- added J3: Conn_01x06, Connector_PinHeader_2.54mm:PinHeader_1x06_P2.54mm_Vertical, F.Cu at (121.0, 85.7)
- added J4: Conn_01x04, Connector_PinHeader_2.54mm:PinHeader_1x04_P2.54mm_Vertical, F.Cu at (244.0, 97.5)
- added R10: 10k, Resistor_SMD:R_0603_1608Metric, F.Cu at (237.3, 78.3)
- added R11: 10k, Resistor_SMD:R_0603_1608Metric, F.Cu at (237.3, 80.8)
- added R12: 100, Resistor_SMD:R_0603_1608Metric, F.Cu at (153.6, 70.2)
- added R13: 330, Resistor_SMD:R_0603_1608Metric, F.Cu at (247.3, 75.8)
- added R14: 100, Resistor_SMD:R_0603_1608Metric, F.Cu at (247.3, 82.8)
- added R15: 100, Resistor_SMD:R_0603_1608Metric, F.Cu at (173.0, 97.9)
- added R16: 100, Resistor_SMD:R_0603_1608Metric, F.Cu at (247.3, 85.3)
- added R17: 100, Resistor_SMD:R_0603_1608Metric, F.Cu at (237.3, 102.5)
- added REN1: 10k, Resistor_SMD:R_0603_1608Metric, F.Cu at (241.3, 70.8)
- added ROFF1: 47k, Resistor_SMD:R_0603_1608Metric, F.Cu at (241.3, 73.3)
- added RRCOFF1: 1k, Resistor_SMD:R_0603_1608Metric, F.Cu at (241.3, 75.8)
- added RSNSA1: 330m, Resistor_SMD:R_0603_1608Metric, F.Cu at (241.3, 78.3)
- added RSNSB1: 330m, Resistor_SMD:R_0603_1608Metric, F.Cu at (241.3, 80.8)
- added U2: HC-SR04, minimouse:HC-SR04, F.Cu at (151.3, 61.9)
- added U3: STSPIN240, Package_DFN_QFN:VQFN-16-1EP_3x3mm_P0.5mm_EP1.8x1.8mm, F.Cu at (132.5, 66.5)
- U4: value HC-SR04 -> LP5907MFX-3.3; footprint minimouse:HC-SR04 -> Package_TO_SOT_SMD:SOT-23-5
- moved R7 21.3 mm to (173.0, 95.3), turned to 180 degrees
- moved C3 19.8 mm to (143.2, 67.0)
- moved C5 11.1 mm to (132.2, 97.5)
- moved J1 10.3 mm to (172.9, 78.3)
- moved R9 9.47 mm to (142.4, 72.9)
- moved R2 6.27 mm to (142.4, 101.7)
- moved R5 4.55 mm to (150.0, 101.7)
- moved R4 3.69 mm to (147.5, 101.7)
- moved R6 3.02 mm to (152.5, 101.7)
- moved R3 2.94 mm to (144.9, 101.7)
- moved C1 2.71 mm to (139.1, 90.2)
Connections:
- R2 pad 2: /mcu/TIM15_CH1 -> /SPIN_PWM_A
- R4 pad 2: /mcu/OUT_A4 -> /SPIN_PH_A
- R7 pad 1: /mcu/OUT_B1 -> /MA_C1
- R7 pad 2: Net-(U1-PB1) -> Net-(J2-Pin_3)
- U1 pad 10: /mcu/TIM2_CH1 -> /MB_C1
- U1 pad 11: /mcu/TIM2_CH2 -> /MB_C2
- U1 pad 16: /mcu/TIM3_CH1 -> /MA_C1
- U1 pad 19: Net-(U1-PB1) -> /SPIN_EN
- U4 pad 1: GND -> +BATT
- U4 pad 2: /mcu/OUT_B9 -> GND
- U4 pad 3: Net-(U4-ECHO) -> +BATT
- U4 pad 4: +3V3 -> unconnected-(U4-NC-Pad4)

Commit message: fin de TP4
Parts:
- moved J4 121.2 mm to (124.6, 76.8)
- moved C13 114.0 mm to (127.4, 77.6), turned to 90 degrees
- moved C8 113.7 mm to (134.6, 95.0), turned to -90 degrees
- moved R17 112.0 mm to (127.4, 80.8), turned to 90 degrees
- moved R16 111.5 mm to (136.2, 95.0), turned to 90 degrees
- moved R14 110.2 mm to (137.8, 95.0), turned to 90 degrees
- moved RSNSB1 99.6 mm to (142.9, 96.5), turned to -90 degrees
- moved C10 99.3 mm to (148.0, 72.0), turned to 180 degrees
- moved ROFF1 98.1 mm to (146.0, 96.4), turned to -90 degrees
- moved RRCOFF1 95.9 mm to (147.6, 96.3), turned to -90 degrees
- moved CRCOFF1 95.1 mm to (144.4, 96.4), turned to -90 degrees
- moved C12 94.6 mm to (148.5, 103.3), turned to -90 degrees
- moved RSNSA1 94.4 mm to (150.3, 103.3), turned to 90 degrees
- moved C11 92.0 mm to (155.4, 68.6), turned to -90 degrees
- moved R13 90.6 mm to (157.0, 68.7), turned to 90 degrees
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Routing:
- net /mcu/~{RESET}: track 0.00 -> 48.2 mm, vias 0 -> 2
- net GND: track 0.00 -> 34.6 mm, vias 0 -> 1
- net +3.3V: track 0.00 -> 21.6 mm
- net /mcu/OUT_B9: track 0.00 -> 14.5 mm
- net Net-(U2-ECHO): track 0.00 -> 6.87 mm
- net /mcu/BOOT0: track 0.00 -> 6.22 mm
- net Net-(U1-PB6): track 0.00 -> 5.72 mm
- net Net-(U1-PB9): track 0.00 -> 5.72 mm
- net +BATT: track 0.00 -> 5.25 mm
- net Net-(D1-A): track 0.00 -> 1.69 mm
- net Net-(U3-REF): track 0.00 -> 1.68 mm
- net /mcu/SWO: track 0.00 -> 0.90 mm
- net /MA_C1: track 0.00 -> 0.77 mm

Commit message: fin TP4
Parts:
- removed R12: 100, Resistor_SMD:R_0603_1608Metric
- moved R7 25.8 mm to (148.7, 90.6)
- moved R15 25.7 mm to (150.3, 90.6), turned to -90 degrees
- moved C9 15.7 mm to (139.0, 82.0), turned to 90 degrees
- moved C5 14.7 mm to (140.8, 82.0), turned to 90 degrees
- moved C3 13.9 mm to (156.7, 85.8), turned to 0 degrees
- moved CRCOFF1 13.8 mm to (158.2, 95.5), turned to 0 degrees
- moved J3 13.2 mm to (126.5, 92.3), turned to 90 degrees
- moved RSNSB1 12.8 mm to (154.8, 101.1), turned to 0 degrees
- moved R16 9.99 mm to (140.9, 86.2), turned to -90 degrees
- moved ROFF1 9.39 mm to (155.0, 93.6), turned to 0 degrees
- moved C7 9.38 mm to (170.3, 89.1), turned to 180 degrees
- moved R14 8.89 mm to (138.8, 86.2), turned to -90 degrees
- moved J4 8.03 mm to (129.9, 82.8), turned to 180 degrees
- moved C1 7.83 mm to (147.3, 73.3), turned to 0 degrees
- moved C13 7.47 mm to (133.4, 82.0), turned to -90 degrees
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Routing:
- net +BATT: track 5.25 -> 57.5 mm
- net +3.3V: track 21.6 -> 53.6 mm
- net /motorA/MB: track 0.00 -> 31.2 mm
- net Net-(J2-Pin_4): track 0.00 -> 26.7 mm, vias 0 -> 2
- net /motorB/MA: track 0.00 -> 25.9 mm
- net Net-(J2-Pin_3): track 0.00 -> 22.3 mm, vias 0 -> 2
- net /motorA/MA: track 0.00 -> 17.1 mm
- net /mcu/IN_B2: track 0.00 -> 14.5 mm
- net GND: track 34.6 -> 49.0 mm, vias 1 -> 15
- net /motorB/MB: track 0.00 -> 14.3 mm, vias 0 -> 3
- net /mcu/SWO: track 0.90 -> 12.4 mm
- net Net-(J3-Pin_3): track 0.00 -> 9.41 mm
- net Net-(J3-Pin_4): track 0.00 -> 8.92 mm
- net /mcu/SWDCLK: track 0.00 -> 8.77 mm
- net /SPIN_PWM_A: track 0.00 -> 8.70 mm
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- added copper zone on B.Cu, net GND
